File: PCB/Microne_PCB.kicad_pcb (KiCad board)
At the start: 2 copper layers, 49 parts, among them J1 Conn_01x24_Male, J2 Conn_01x02_Male, J3 Conn_01x02_Male, J4 Conn_01x02_Male, J5 Conn_01x02_Male, J6 Conn_01x02_Male, J7 Conn_01x02_Male, J8 Conn_01x05_Male, K1 FINDER-36.11, K2 FINDER-36.11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

Commit message: PCB Prototype
Parts:
- removed C1, C2, C4: 4.7u, Capacitor_SMD:C_0603_1608Metric
- removed C6: 1u, Capacitor_SMD:C_0603_1608Metric
- removed C7: 10u, Capacitor_SMD:C_0603_1608Metric
- removed R1: 1M, Resistor_SMD:R_0201_0603Metric
- removed R14, R15, R16, R3, R4, R5: 4.7k, Resistor_SMD:R_0201_0603Metric
- removed R2: 10k, Resistor_SMD:R_0201_0603Metric
- added J10: Conn_01x02_Male, Connector_Phoenix_MSTB:PhoenixContact_MSTBVA_2,5_2-G_1x02_P5.00mm_Vertical, F.Cu at (205.4, 92.4)
- added J9: Conn_01x02_Male, Connector_PinHeader_2.54mm:PinHeader_1x02_P2.54mm_Vertical, F.Cu at (161.2, 66.9)
- D1, D2, D3, D4: moved to B.Cu
- J1: value Conn_01x24_Male -> Conn_02x20_Odd_Even; footprint Connector_FFC-FPC:Hirose_FH12-24S-0.5SH_1x24-1MP_P0.50mm_Horizontal -> Connector_PinHeader_2.54mm:PinHeader_2x20_P2.54mm_Vertical; moved to F.Cu
- J8: value Conn_01x05_Male -> Conn_01x03_Male; footprint Connector_PinHeader_2.54mm:PinHeader_1x05_P2.54mm_Vertical -> Connector_PinHeader_2.54mm:PinHeader_1x03_P2.54mm_Vertical
- moved Q4 362.5 mm to (198.9, 117.6)
- moved R9 360.7 mm to (198.8, 113.0), turned to -90 degrees
- moved Q3 340.4 mm to (187.9, 117.6)
- moved J7 336.1 mm to (198.5, 132.0)
- moved R8 333.2 mm to (188.0, 113.2), turned to -90 degrees
- moved J5 321.1 mm to (171.3, 132.0)
- moved Q1 311.1 mm to (193.6, 107.7), turned to -90 degrees
- moved J6 310.2 mm to (184.9, 132.0)
- moved J4 304.4 mm to (153.9, 132.0)
- moved Q2 295.7 mm to (188.6, 107.7), turned to -90 degrees
- moved R10 292.8 mm to (198.7, 123.0), turned to -90 degrees
- moved U1 290.5 mm to (155.5, 72.8), turned to -90 degrees
- moved Q5 287.3 mm to (193.0, 121.6), turned to -90 degrees
- moved R13 284.7 mm to (201.2, 113.0), turned to 90 degrees
- moved Q8 281.1 mm to (198.6, 107.7), turned to -90 degrees
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Connections:
- J1 pad 10: /DC -> unconnected-(J1-Pad10)
- J1 pad 11: GND -> unconnected-(J1-Pad11)
- J1 pad 12: GND -> unconnected-(J1-Pad12)
- J1 pad 13: /CLK -> unconnected-(J1-Pad13)
- J1 pad 14: /DIN -> GND
- J1 pad 15: /BS2 -> unconnected-(J1-Pad15)
- J1 pad 16: GND -> unconnected-(J1-Pad16)
- J1 pad 17: GND -> unconnected-(J1-Pad17)
- J1 pad 18: GND -> /DC
- J1 pad 19: GND -> /DIN
- J1 pad 2: GND -> +3.3V
- J1 pad 21: Net-(J1-Pad21) -> unconnected-(J1-Pad21)
- J1 pad 22: Net-(J1-Pad22) -> /RST
- J1 pad 23: +12V -> /CLK
- J1 pad 24: unconnected-(J1-Pad24) -> /CS
- J1 pad 3: GND -> unconnected-(J1-Pad3)
- J1 pad 4: unconnected-(J1-Pad4) -> +3.3V
- J1 pad 5: +3.3V -> unconnected-(J1-Pad5)
- J1 pad 6: /BS1 -> GND
- J1 pad 7: GND -> unconnected-(J1-Pad7)
- J1 pad 8: /CS -> unconnected-(J1-Pad8)
- J1 pad 9: /RST -> unconnected-(J1-Pad9)
- J8 pad 1: +3.3V -> /ENC_B
- J8 pad 2: GND -> /ENC_A
- J8 pad 3: /ENC_A -> /ENC_SW
- K1 pad 14: +12V -> VDC
- K2 pad 14: +12V -> VDC
- K3 pad 14: +12V -> VDC
- K4 pad 14: +12V -> VDC
- Q1 pad 1: +12V -> VDC
- Q2 pad 1: +12V -> VDC
- R12 pad 1: /RELAY_1 -> /RELAY_2
- R13 pad 1: /RELAY_2 -> /RELAY_3
- R8 pad 1: +12V -> VDC
- R9 pad 1: +12V -> VDC
Routing:
- net +3.3V: track 0.00 -> 173.7 mm
- net Net-(Q1-Pad2): track 0.00 -> 157.8 mm, vias 0 -> 3
- net /RELAY_0: track 0.00 -> 150.1 mm, vias 0 -> 2
- net /RELAY_1: track 0.00 -> 148.1 mm, vias 0 -> 2
- net Net-(Q2-Pad2): track 0.00 -> 146.2 mm, vias 0 -> 1
- net VDC: track 0.00 -> 118.8 mm
- net /RELAY_2: track 0.00 -> 100.3 mm, vias 0 -> 2
- net /RELAY_3: track 0.00 -> 93.3 mm, vias 0 -> 4
- net Net-(D1-Pad2): track 0.00 -> 84.8 mm
- net /CS: track 0.00 -> 77.5 mm
- net /RST: track 0.00 -> 71.1 mm
- net /DIN: track 0.00 -> 69.2 mm
- net /CLK: track 0.00 -> 68.0 mm
- net Net-(D3-Pad2): track 0.00 -> 67.7 mm
- net /DC: track 0.00 -> 62.9 mm
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- added copper zone on B.Cu, net GND
- added copper zone on B.Cu, net VDC
Other:
- board outline added: 96 x 88 mm
- board text added: "3V3"
- board text added: "GND"
- board text added: "PWM0"
- board text added: "PWM1"
- board text removed: "SCREEN"
