File: PCB/Microne_PCB.kicad_sch (KiCad schematic)
At the start: 33 parts, among them J1 Conn_01x24_Male, J2 Conn_01x02_Male, J3 Conn_01x02_Male, J4 Conn_01x02_Male, J5 Conn_01x02_Male, J6 Conn_01x02_Male, J7 Conn_01x02_Male, J8 Conn_01x05_Male, Q1 BC547, Q2 BC547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

Commit message: PCB Prototype
Parts:
- removed C1, C2, C4: 4.7u, Capacitor_SMD:C_0603_1608Metric, symbol Device:C
- removed C6: 1u, Capacitor_SMD:C_0603_1608Metric, symbol Device:C
- removed C7: 10u, Capacitor_SMD:C_0603_1608Metric, symbol Device:C
- removed J1: Conn_01x24_Male, Connector_FFC-FPC:Hirose_FH12-24S-0.5SH_1x24-1MP_P0.50mm_Horizontal, symbol Connector:Conn_01x24_Male
- removed J8: Conn_01x05_Male, Connector_PinHeader_2.54mm:PinHeader_1x05_P2.54mm_Vertical, symbol Connector:Conn_01x05_Male
- removed R1: 1M, Resistor_SMD:R_0201_0603Metric, symbol Device:R
- removed R14, R15, R16, R3, R4, R5: 4.7k, Resistor_SMD:R_0201_0603Metric, symbol Device:R
- removed R2: 10k, Resistor_SMD:R_0201_0603Metric, symbol Device:R
- added J1: Conn_02x20_Odd_Even, Connector_PinHeader_2.54mm:PinHeader_2x20_P2.54mm_Vertical, symbol Connector_Generic:Conn_02x20_Odd_Even
- added J10: Conn_01x02_Male, Connector_Phoenix_MSTB:PhoenixContact_MSTBVA_2,5_2-G_1x02_P5.00mm_Vertical, symbol Connector:Conn_01x02_Male
- added J8: Conn_01x03_Male, Connector_PinHeader_2.54mm:PinHeader_1x03_P2.54mm_Vertical, symbol Connector:Conn_01x03_Male
- added J9: Conn_01x02_Male, Connector_PinHeader_2.54mm:PinHeader_1x02_P2.54mm_Vertical, symbol Connector:Conn_01x02_Male
Connections:
- net +12V: no longer Q1.1 (C), Q2.1 (C), R8.1, R9.1
- net +3.3V: now also J1.2 (Pin_2), J1.4 (Pin_4), J9.2 (Pin_2)
- net CLK: now also J1.23 (Pin_23)
- net CS: now also J1.24 (Pin_24)
- net DC: now also J1.18 (Pin_18)
- net DIN: now also J1.19 (Pin_19)
- net ENC_A: now also J8.2 (Pin_2)
- net ENC_B: now also J8.1 (Pin_1)
- net ENC_SW: now also J8.3 (Pin_3)
- net GND: now also J1.14 (Pin_14), J1.20 (Pin_20), J1.25 (Pin_25), J1.30 (Pin_30), J1.34 (Pin_34), J1.39 (Pin_39), J1.6 (Pin_6), J10.1 (Pin_1), J9.1 (Pin_1)
- net RST: now also J1.22 (Pin_22)
- net VDC: now also Q1.1 (C), Q2.1 (C), R8.1, R9.1, J10.2 (Pin_2)
- no-connect marks 23 -> 46
