File: PCB/untitled.kicad_sch (KiCad schematic)
At the start: 4 parts, among them K1 FINDER-36.11, Q5 BC547

Commit message: PCB Prototype
Connections:
- net +12V renamed VDC
Changed lines of the file:
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@@
     (pin "A2")
   )
-  (symbol (lib_id "power:+12V") (at 137.16 69.85 0) (unit 1)
+  (symbol (lib_id "power:VDC") (at 137.16 69.85 0) (unit 1)
     (in_bom yes) (on_board yes) (fields_autoplaced)
-    (property "Reference" "#PWR015" (id 0) (at 137.16 73.66 0)
+    (property "Reference" "#PWR0101" (id 0) (at 137.16 72.39 0)
       (effects (font (size 1.27 1.27)) hide)
     )
-    (property "Value" "+12V" (id 1) (at 137.16 64.77 0))
+    (property "Value" "VDC" (id 1) (at 137.16 64.77 0))
     (property "Footprint" "" (id 2) (at 137.16 69.85 0)
       (effects (font (size 1.27 1.27)) hide)
